File: pcb/wingboard.kicad_pcb (KiCad board)
At the start: 2 copper layers, 250.3 x 147.1 mm, 109 parts

Commit message: Updated pcb
Parts:
- moved S3 1.68 mm to (71.3, 78.9)
- moved D43 1.68 mm to (210.4, 116.7)
- moved S47 1.68 mm to (207.2, 157.9)
- moved S45 1.68 mm to (197.1, 80.1)
- moved S46 1.68 mm to (227.6, 143.5)
- moved S17 1.68 mm to (136.6, 72.0)
- moved D19 1.68 mm to (139.5, 116.7)
- moved S43 1.68 mm to (208.7, 112.0)
- moved D45 1.68 mm to (198.8, 84.8)
- moved S21 1.68 mm to (152.8, 80.1)
- moved S48 1.68 mm to (195.0, 179.7)
- moved D34 1.68 mm to (247.4, 112.9)
- moved S2 1.68 mm to (66.9, 95.3)
- moved S5 1.68 mm to (85.7, 106.7)
- moved H2 1.68 mm to (80.3, 121.5)
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Routing:
- net P006: track 0.00 -> 157.4 mm, vias 0 -> 2
- net P113: track 0.00 -> 155.5 mm, vias 0 -> 2
- net P111: track 0.00 -> 155.2 mm
- net P010: track 0.00 -> 143.2 mm
- net P009: track 0.00 -> 133.4 mm
- net P115: track 0.00 -> 133.1 mm
- net P104: track 0.00 -> 132.1 mm
- net P008: track 0.00 -> 131.6 mm
- net P002: track 0.00 -> 125.6 mm
- net P017: track 0.00 -> 118.7 mm
- net P029: track 0.00 -> 107.3 mm
- net P020: track 0.00 -> 95.9 mm
- net P022: track 0.00 -> 69.4 mm
- net P031: track 0.00 -> 69.4 mm
- net P106: track 0.00 -> 58.9 mm
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
Commit message: More PCB routing changes
Parts:
- moved D44 0.94 mm to (205.6, 100.6)
- moved S3 0.94 mm to (72.2, 78.8)
- moved S46 0.94 mm to (228.6, 143.4)
- moved D45 0.94 mm to (199.7, 84.7)
- moved S47 0.94 mm to (208.2, 157.8)
- moved S5 0.94 mm to (86.6, 106.6)
- moved S21 0.94 mm to (153.8, 80.0)
- moved S42 0.94 mm to (215.5, 127.9)
- moved D43 0.94 mm to (211.4, 116.6)
- moved S27 0.94 mm to (279.6, 78.8)
- moved S45 0.94 mm to (198.0, 80.0)
- moved D33 0.94 mm to (254.1, 128.7)
- moved S10 0.94 mm to (105.2, 108.1)
- moved RE1 0.94 mm to (175.9, 161.8)
- moved S12 0.94 mm to (116.8, 76.1)
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Connections:
- S25 pad 1: P022 -> P006
- S26 pad 1: P022 -> P006
- S27 pad 1: P022 -> P006
- S28 pad 1: P022 -> P006
- S29 pad 1: P020 -> P008
- S30 pad 1: P020 -> P008
- S31 pad 1: P020 -> P008
- S32 pad 1: P020 -> P008
- S33 pad 1: P020 -> P008
- S38 pad 1: P008 -> P020
- S39 pad 1: P008 -> P020
- S40 pad 1: P008 -> P020
- S41 pad 1: P008 -> P020
- S42 pad 1: P006 -> P022
- S43 pad 1: P006 -> P022
- S44 pad 1: P006 -> P022
- S45 pad 1: P006 -> P022
- S47 pad 1: P008 -> P020
- S48 pad 1: P006 -> P022
Routing:
- net P106: track 58.9 -> 344.9 mm, vias 0 -> 1
- net P104: track 132.1 -> 375.5 mm, vias 0 -> 2
- net P009: track 133.4 -> 355.8 mm
- net P010: track 143.2 -> 347.7 mm, vias 0 -> 2
- net P111: track 155.2 -> 359.5 mm, vias 0 -> 2
- net P024: track 0.00 -> 146.5 mm, vias 0 -> 2
- net P100: track 0.00 -> 142.9 mm, vias 0 -> 2
- net P022: track 69.4 -> 162.7 mm, vias 0 -> 2
- net P020: track 95.9 -> 173.9 mm
- net P017: track 118.7 -> 174.2 mm
- net ring_r2: track 14.2 -> 56.5 mm
- net P008: track 131.6 -> 171.6 mm
- net VCC: track 0.00 -> 27.3 mm, vias 0 -> 1
- net P006: track 157.4 -> 174.4 mm, vias 2 -> 0
- net P115: track 133.1 -> 143.9 mm
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
Commit message: Updated the PCB
Parts:
- moved S13 1.05 mm to (123.5, 60.8)
- moved S19 1.05 mm to (143.0, 112.6)
- moved H4 1.05 mm to (176.7, 180.2)
- moved MCU1 1.05 mm to (176.7, 91.6)
- moved D22 1.05 mm to (122.4, 148.7)
- moved S17 1.05 mm to (138.4, 72.6)
- moved S33 1.05 mm to (253.2, 124.7)
- moved D26 1.05 mm to (286.1, 100.7)
- moved S18 1.05 mm to (137.1, 128.5)
- moved S7 1.05 mm to (99.1, 75.3)
- moved S28 1.05 mm to (276.0, 63.0)
- moved S35 1.05 mm to (241.6, 92.7)
- moved S26 1.05 mm to (284.8, 95.8)
- moved D3 1.05 mm to (71.8, 84.2)
- moved D35 1.05 mm to (243.3, 97.4)
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Connections:
- RE1 pad S1: (no net) -> P011
- RE1 pad S2: (no net) -> GND
Routing:
- net P011: track 0.00 -> 128.1 mm, vias 0 -> 5
- net P031: track 76.6 -> 192.4 mm
- net P029: track 115.2 -> 203.2 mm, vias 0 -> 2
- net BAT_P: track 0.00 -> 81.6 mm, vias 0 -> 1
- net RST: track 0.00 -> 58.8 mm
- net P002: track 136.4 -> 186.3 mm, vias 0 -> 2
- net RAW: track 0.00 -> 40.1 mm
- net ring_r2: track 56.5 -> 16.4 mm
- net P115: track 143.9 -> 176.7 mm, vias 0 -> 2
- net P113: track 164.9 -> 180.8 mm, vias 2 -> 4
- net P009: track 355.8 -> 348.5 mm
- net inner_r3: track 18.5 -> 24.0 mm
- net P104: track 375.5 -> 371.3 mm
- net P022: track 162.7 -> 165.1 mm
- net P010: track 347.7 -> 345.6 mm
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- added copper zone on B.Cu, net GND
- added copper zone on F.Cu, net GND

Commit message: Updated PCB and config
Parts:
- moved D39 1.15 mm to (228.6, 108.1)
- moved S45 1.15 mm to (199.0, 79.5)
- moved H2 1.15 mm to (82.2, 120.9)
- moved S17 1.15 mm to (138.5, 71.4)
- moved S33 1.15 mm to (253.4, 123.5)
- moved S13 1.15 mm to (123.6, 59.6)
- moved S19 1.15 mm to (143.1, 111.4)
- moved D12 1.15 mm to (116.1, 80.3)
- moved S11 1.15 mm to (112.0, 91.6)
- moved S3 1.15 mm to (73.2, 78.3)
- moved D44 1.15 mm to (206.5, 100.1)
- moved S7 1.15 mm to (99.2, 74.2)
- moved S21 1.15 mm to (154.7, 79.5)
- moved D29 1.15 mm to (267.9, 110.8)
- moved RST1 1.15 mm to (213.8, 57.4)
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Routing:
- net GND: track 0.00 -> 37.0 mm, vias 0 -> 1
- net P010: track 345.6 -> 336.2 mm
- net P101: track 0.00 -> 5.84 mm
- net P020: track 173.9 -> 170.1 mm
- net P104: track 371.3 -> 374.2 mm
- net ring_r4: track 18.5 -> 16.4 mm
- net inner_r4: track 18.5 -> 16.4 mm
- net mirror_middle_r5: track 18.5 -> 16.4 mm
- net middle_r4: track 18.5 -> 16.4 mm
- net index_r4: track 18.5 -> 16.4 mm
- net P008: track 171.6 -> 170.4 mm
- net P017: track 174.2 -> 173.1 mm
- net P111: track 359.5 -> 360.7 mm
- net P009: track 348.5 -> 349.4 mm
Other:
- outline, holes or cut-outs redrawn

Commit message: Updated PCB, added new image footprint, and updated config
Parts:
- added G***: LOGO, wingboard.kicad_pro:Wingboard logo, F.Cu at (176.5, 163.5)
- added G***: LOGO, wingboard.kicad_pro:Wingboard logo, F.Cu at (176.6, 163.3)
- added G***: LOGO, wingboard.kicad_pro:Wingboard logo, F.Cu at (176.7, 163.2)
- moved S33 0.69 mm to (253.1, 124.2)
- moved D2 0.69 mm to (67.3, 100.2)
- moved S45 0.69 mm to (198.8, 80.1)
- moved S21 0.69 mm to (154.5, 80.1)
- moved S9 0.69 mm to (100.2, 124.2)
- moved S11 0.69 mm to (111.8, 92.2)
- moved D27 0.69 mm to (281.6, 83.7)
- moved S7 0.69 mm to (99.0, 74.8)
- moved D29 0.69 mm to (267.7, 111.5)
- moved D47 0.69 mm to (212.6, 161.3)
- moved S1 0.69 mm to (64.2, 111.8)
- moved S37 0.69 mm to (229.9, 60.3)
- moved D1 0.69 mm to (62.9, 116.6)
- moved S34 0.69 mm to (247.3, 108.2)
- moved T1 0.69 mm to (139.7, 58.0)
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Routing:
- net GND: track 37.0 -> 37.7 mm
Other:
- board text added: "Back"
- board text added: "Front"
- board text added: "Nice!View goes here"
- board text added: "Supermini NRF52840 goes here"

Commit message: Added new footprints, updated PCB and config
Parts:
- removed JST1: , ceoloide:battery_connector_jst_ph_2
- removed RST1: , ceoloide:reset_switch_smd_side
- removed T1: , E73:SPDT_C128955
- added JSTPH2: JST_PH_S2B-PH-SM4-TB_1x02-1MP_P2.00mm_Horizontal, Connector_JST:JST_PH_S2B-PH-SM4-TB_1x02-1MP_P2.00mm_Horizontal, B.Cu at (191.4, 103.8)
- added PWR: SW_SPDT_PCM12, Button_Switch_SMD:SW_SPDT_PCM12, B.Cu at (139.6, 58.2)
- added RST: Panasonic_EVQPUL_EVQPUC, Button_Switch_SMD:Panasonic_EVQPUL_EVQPUC, B.Cu at (213.6, 58.1)
