File: pcb/wingboard.kicad_pcb (KiCad board)
At the start: 2 copper layers, 250.3 x 147.1 mm, 112 parts

Commit message: Created Production PCB and updated Readme
Parts:
- removed the G*** at (176.5, 163.5)
- removed the G*** at (176.6, 163.3)
- removed the G*** at (176.7, 163.2)
- removed JSTPH2: JST_PH_S2B-PH-SM4-TB_1x02-1MP_P2.00mm_Horizontal, Connector_JST:JST_PH_S2B-PH-SM4-TB_1x02-1MP_P2.00mm_Horizontal
- removed PWR: SW_SPDT_PCM12, Button_Switch_SMD:SW_SPDT_PCM12
- removed RST: Panasonic_EVQPUL_EVQPUC, Button_Switch_SMD:Panasonic_EVQPUL_EVQPUC
- added G***: LOGO, wingboard.kicad_pro:Wingboard logo, F.Cu at (191.1, 154.9)
- added JST_BAT1: JST_PH_S2B-PH-SM4-TB_1x02-1MP_P2.00mm_Horizontal, Connector_JST:JST_PH_S2B-PH-SM4-TB_1x02-1MP_P2.00mm_Horizontal, B.Cu at (206.4, 97.4)
- added PWR1: SW_SPDT_PCM12, Button_Switch_SMD:SW_SPDT_PCM12, B.Cu at (153.9, 49.5)
- added RST1: Panasonic_EVQPUL_EVQPUC, Button_Switch_SMD:Panasonic_EVQPUL_EVQPUC, B.Cu at (227.7, 49.7)
- D1, D10, D11, D12, D13, D14, D15, D16, D17, D18, D19, D2, D20, D21, D22, D23, D24, D25, D26, D27, D28, D29, D3, D30, D31, D32, D33, D34, D35, D36, D37, D38, D39, D4, D40, D41, D42, D43, D44, D45, D46, D47, D48, D5, D6, D7, D8, D9: footprint ComboDiode -> ceoloide:diode_tht_sod123; moved to B.Cu
- moved S37 16.5 mm to (244.0, 51.8)
- moved S11 16.5 mm to (125.9, 83.8)
- moved S19 16.5 mm to (157.0, 103.6)
- moved MCU1 16.5 mm to (190.8, 82.6)
- moved S40 16.5 mm to (235.0, 79.6)
- moved D7 16.5 mm to (111.4, 71.0)
- moved S33 16.5 mm to (267.3, 115.7)
- moved S44 16.5 mm to (218.8, 87.6)
- moved D22 16.5 mm to (136.4, 139.7)
- moved D30 16.5 mm to (276.0, 87.0)
- moved S43 16.5 mm to (224.6, 103.6)
- moved D18 16.5 mm to (149.5, 124.3)
- moved S22 16.5 mm to (138.1, 135.0)
- moved D46 16.5 mm to (245.2, 139.7)
- moved S48 16.5 mm to (210.9, 171.2)
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Routing:
- net P010: track 336.2 -> 277.7 mm, vias 2 -> 12
- net P111: track 360.7 -> 303.6 mm, vias 2 -> 12
- net P009: track 349.4 -> 294.2 mm, vias 0 -> 10
- net P104: track 374.2 -> 329.7 mm, vias 2 -> 12
- net P106: track 344.9 -> 306.1 mm, vias 1 -> 9
- net inner_r3: track 24.0 -> 20.0 mm
- net BAT_P: track 81.6 -> 84.5 mm
- net P011: track 128.1 -> 130.5 mm
- net index_r4: track 16.4 -> 14.2 mm
- net home_thumb: track 15.8 -> 13.6 mm
- net ring_r3: track 16.4 -> 14.2 mm
- net mirror_middle_r3: track 16.4 -> 14.2 mm
- net mirror_index_r4: track 16.4 -> 14.2 mm
- net inner_r2: track 16.4 -> 14.2 mm
- net middle_r2: track 16.4 -> 14.2 mm
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Other:
- board text added: "+"
- board text added: "-"
